Commit message: Geometry of depth camera updated.

File: robots/mpo_700/xacros/depth_camera.xacro (robot description, xacro)
@@ -17,5 +17,5 @@
 			    </collision>
 			    <visual>
-			      <origin xyz="0 0 0" rpy="1.570796 0 1.570796"/>
+			      <origin xyz="0 -0.0175 0" rpy="1.570796 0 1.570796"/>
 			      <geometry>
 			      	<mesh filename="package://neo_simulation/robots/mpo_700/meshes/d435.dae"/>
