Commit message: Robot model of mpo_700 updated, RealSense D435i included.

File: robots/mpo_700/mpo_700.urdf.xacro (robot description, xacro)
@@ -14,4 +14,5 @@
   <xacro:include filename="$(find neo_simulation)/robots/mpo_700/xacros/ultrasonic.xacro" />
   <-->
+  <xacro:include filename="$(find neo_simulation)/robots/mpo_700/xacros/depth_camera.xacro" />
   <!--Gazebo  -->
   <xacro:include filename="$(find neo_simulation)/robots/mpo_700/xacros/mpo_700_gazebo.xacro" />
@@ -137,3 +138,13 @@
   </xacro:camera>
   <-->
+  <xacro:depth_camera name="camera" parent="base_link">
+    <origin xyz="0.25 0 0.45" rpy="0 0 0" />
+  </xacro:depth_camera>
+  <joint name="camera_optical_joint" type="fixed">
+    <origin xyz="0 0 0" rpy="${-pi/2} 0 ${-pi/2}"/>
+    <parent link="camera_link"/>
+    <child link="camera_link_optical"/>
+  </joint>
+  <link name="camera_link_optical">
+  </link>
 </robot>

File: robots/mpo_700/xacros/camera.xacro (robot description, xacro)
@@ -9,4 +9,13 @@
     </joint>
     <link name="${name}_link">
+      <visual>
+        <origin xyz="0 0 0" rpy="0 0 0"/>
+        <geometry>
+        <box size="0.05 0.05 0.05"/>
+        </geometry>
+        <material name="red">
+          <color rgba="1 0 0 1" />
+        </material>
+      </visual>
       <inertial>
         <mass value="0.001" />

File: robots/mpo_700/xacros/mpo_700_gazebo.xacro (robot description, xacro)
@@ -104,4 +104,5 @@
   </gazebo>
   <!-- camera -->
+  <!-->
   <gazebo reference="camera_link">
     <sensor type="camera" name="camera1">
@@ -120,7 +121,7 @@
         <noise>
           <type>gaussian</type>
-          <!-- Noise is sampled independently per pixel on each frame.
+           Noise is sampled independently per pixel on each frame.
                That pixel's noise value is added to each of its color
-               channels, which at that point lie in the range [0,1]. -->
+               channels, which at that point lie in the range [0,1].
           <mean>0.0</mean>
           <stddev>0.007</stddev>
@@ -140,4 +141,35 @@
         <distortionT1>0.0</distortionT1>
         <distortionT2>0.0</distortionT2>
+      </plugin>
+    </sensor>
+  </gazebo>
+  <-->
+  <gazebo reference="camera_link">
+    <sensor name="camera1" type="depth">
+      <update_rate>15</update_rate>
+      <hfov>70</hfov>
+      <plugin name="camera1_controller" filename="libgazebo_ros_openni_kinect.so">
+        <!--<baseline>0.2</baseline>-->
+        <alwaysOn>true</alwaysOn>
+        <updateRate>0.0</updateRate>
+        <cameraName>camera1_ir</cameraName>
+        <imageTopicName>/camera1/depth/image_raw</imageTopicName>
+        <cameraInfoTopicName>/camera1/depth/camera_info</cameraInfoTopicName>
+        <depthImageTopicName>/camera1depth/depth_raw</depthImageTopicName>
+        <depthImageInfoTopicName>/camera1/depth/camera_info</depthImageInfoTopicName>
+        <pointCloudTopicName>/camera1/depth/points</pointCloudTopicName>
+        <frameName>camera_link_optical</frameName>
+        <pointCloudCutoff>0.12</pointCloudCutoff>
+        <pointCloudCutoffMax>3.0</pointCloudCutoffMax>
+        <distortionK1>0.00000001</distortionK1>
+        <distortionK2>0.00000001</distortionK2>
+        <distortionK3>0.00000001</distortionK3>
+        <distortionT1>0.00000001</distortionT1>
+        <distortionT2>0.00000001</distortionT2>
+        <CxPrime>0</CxPrime>
+        <Cx>0</Cx>
+        <Cy>0</Cy>
+        <focalLength>0</focalLength>
+        <hackBaseline>0</hackBaseline>
       </plugin>
     </sensor>

File: robots/mpo_700/xacros/mpo_700_wheel.xacro (robot description, xacro)
@@ -15,6 +15,6 @@
       <origin xyz="0 0 0" rpy="0 0 0" />
         <inertia  ixx="0.04" ixy="0.000" ixz="0.0"
-                  iyy="0.02" iyz="0.00"
-                  izz="0.05" />
+                  iyy="0.04" iyz="0.00"
+                  izz="0.04" />
     </inertial>
     <visual>

Commit message: Unified topics in simulation and robot, updated geometric size.

File: robots/mpo_700/mpo_700.urdf.xacro (robot description, xacro)
@@ -139,5 +139,5 @@
   <-->
   <xacro:depth_camera name="camera" parent="base_link">
-    <origin xyz="0.25 0 0.45" rpy="0 0 0" />
+    <origin xyz="0.228 0 0.461" rpy="0 0 0" />
   </xacro:depth_camera>
   <joint name="camera_optical_joint" type="fixed">

File: robots/mpo_700/xacros/mpo_700_gazebo.xacro (robot description, xacro)
@@ -172,10 +172,10 @@
         <alwaysOn>true</alwaysOn>
         <updateRate>0.0</updateRate>
-        <cameraName>camera1_ir</cameraName>
-        <imageTopicName>/camera1/depth/image_raw</imageTopicName>
-        <cameraInfoTopicName>/camera1/depth/camera_info</cameraInfoTopicName>
-        <depthImageTopicName>/camera1depth/depth_raw</depthImageTopicName>
-        <depthImageInfoTopicName>/camera1/depth/camera_info</depthImageInfoTopicName>
-        <pointCloudTopicName>/camera1/depth/points</pointCloudTopicName>
+        <cameraName>camera_ir</cameraName>
+        <imageTopicName>/camera/depth/image_raw</imageTopicName>
+        <cameraInfoTopicName>/camera/depth/camera_info</cameraInfoTopicName>
+        <depthImageTopicName>/camera/depth/depth_raw</depthImageTopicName>
+        <depthImageInfoTopicName>/camera/depth/camera_info</depthImageInfoTopicName>
+        <pointCloudTopicName>/camera/depth_registered/points</pointCloudTopicName>
         <frameName>camera_link_optical</frameName>
         <pointCloudCutoff>0.12</pointCloudCutoff>
